Commit message: Scale limo_ackerman robot model to 2x and adjust lane tracking parameters

File: src/limo_description/urdf/limo_ackerman.xacro (robot description, xacro)
@@ -8,25 +8,25 @@
     <xacro:property name="M_PI" value="3.14159"/>
     <!-- Vehicle Geometries -->
-    <xacro:property name="base_x_size" value="0.13" />
-    <xacro:property name="base_y_size" value="0.12" />
-    <xacro:property name="base_z_size" value="0.10" />
-    <xacro:property name="wheelbase" value="0.2"/>
-    <xacro:property name="track" value="0.14"/>
-    <xacro:property name="wheel_vertical_offset" value="-0.100998" />
+    <xacro:property name="base_x_size" value="0.26" />
+    <xacro:property name="base_y_size" value="0.24" />
+    <xacro:property name="base_z_size" value="0.20" />
+    <xacro:property name="wheelbase" value="0.4"/>
+    <xacro:property name="track" value="0.28"/>
+    <xacro:property name="wheel_vertical_offset" value="-0.201996" />
     <xacro:property name="base_mass" value="2.1557"/>
-    <xacro:property name="wheel_length" value="0.045" />
-    <xacro:property name="wheel_radius" value="0.045" />
+    <xacro:property name="wheel_length" value="0.09" />
+    <xacro:property name="wheel_radius" value="0.09" />
     <link name="base_footprint"/>
     <joint name="base_joint" type="fixed">
     <parent link="base_footprint"/>
     <child link="base_link"/>
-    <origin xyz="0.0 0.0 0.15" rpy="0 0 0"/>
+    <origin xyz="0.0 0.0 0.30" rpy="0 0 0"/>
     </joint>
     <!-- Base link -->
     <link name="base_link">
         <visual>
-            <origin xyz="0 0 -0.15" rpy="0 0 1.57" />
+            <origin xyz="0 0 -0.30" rpy="0 0 1.57" />
             <geometry>
-                <mesh filename="package://limo_description/meshes/limo_base.dae" scale="1 1 1"/>
+                <mesh filename="package://limo_description/meshes/limo_base.dae" scale="2 2 2"/>
             </geometry>
         </visual>
@@ -53,11 +53,11 @@
     </joint>
     <xacro:limo_laser parent_prefix="base_link" frame_prefix="laser">
-        <origin xyz="0.103 0 -0.034" rpy="0 0 0"/>
+        <origin xyz="0.206 0 -0.068" rpy="0 0 0"/>
     </xacro:limo_laser>
     <xacro:limo_depth_camera parent_prefix="base_link" frame_prefix="depth_camera">
-        <origin xyz="0.084 0 0.03" rpy="0 0.2618 0"/>
+        <origin xyz="0.168 0 0.06" rpy="0 0.2618 0"/>
     </xacro:limo_depth_camera>
     <xacro:limo_imu parent_prefix="base_link" frame_prefix="imu">
-        <origin xyz="0.0 0 -0.1" rpy="0 0 0"/>
+        <origin xyz="0.0 0 -0.2" rpy="0 0 0"/>
     </xacro:limo_imu>
     <xacro:limo_left_steering_hinge parent_prefix="base_link" wheel_prefix="left_steering_hinge">
@@ -76,5 +76,5 @@
             <origin xyz="0 0 0" rpy="0 0 0" />
             <geometry>
-                <mesh filename="package://limo_description/meshes/limo_wheel.dae" />
+                <mesh filename="package://limo_description/meshes/limo_wheel.dae" scale="2 2 2" />
             </geometry>
         </visual>
@@ -101,5 +101,5 @@
             <origin xyz="0 0 0" rpy="0 0 0" />
             <geometry>
-                <mesh filename="package://limo_description/meshes/limo_wheel.dae" />
+                <mesh filename="package://limo_description/meshes/limo_wheel.dae" scale="2 2 2" />
             </geometry>
         </visual>

File: src/limo_description/urdf/limo_steering_hinge.xacro (robot description, xacro)
@@ -11,5 +11,5 @@
                 <origin xyz="0 0 0" rpy="0 0 0" />
                 <geometry>
-                  <cylinder length="0.0001" radius="0.0001" />
+                  <cylinder length="0.0002" radius="0.0002" />
                 </geometry>
             </visual>
@@ -17,5 +17,5 @@
               <origin xyz="0 ${wheel_length/2} 0" rpy="1.57 0 0" />
               <geometry>
-                  <cylinder length="${wheel_length}" radius="${wheel_radius-0.01}" />
+                  <cylinder length="${wheel_length}" radius="${wheel_radius-0.02}" />
               </geometry>
             </collision>
@@ -38,5 +38,5 @@
               <origin xyz="0 0 0" rpy="0 0 0" />
               <geometry>
-                  <mesh filename="package://limo_description/meshes/limo_wheel.dae" />
+                  <mesh filename="package://limo_description/meshes/limo_wheel.dae" scale="2 2 2" />
               </geometry>
           </visual>
@@ -65,5 +65,5 @@
                 <origin xyz="0 0 0" rpy="0 0 0" />
                 <geometry>
-                  <cylinder length="0.0001" radius="0.0001" />
+                  <cylinder length="0.0002" radius="0.0002" />
                 </geometry>
             </visual>
@@ -71,5 +71,5 @@
               <origin xyz="0 ${wheel_length/2} 0" rpy="1.57 0 0" />
               <geometry>
-                  <cylinder length="${wheel_length}" radius="${wheel_radius-0.01}" />
+                  <cylinder length="${wheel_length}" radius="${wheel_radius-0.02}" />
               </geometry>
             </collision>
@@ -92,5 +92,5 @@
               <origin xyz="0 0 0" rpy="0 0 0" />
               <geometry>
-                  <mesh filename="package://limo_description/meshes/limo_wheel.dae" />
+                  <mesh filename="package://limo_description/meshes/limo_wheel.dae" scale="2 2 2" />
               </geometry>
           </visual>

File: src/limo_description/urdf/limo_xacro.xacro (robot description, xacro)
@@ -11,5 +11,5 @@
                 <origin xyz="0 0 0" rpy="0 0 0" />
                 <geometry>
-                    <mesh filename="package://limo_description/meshes/limo_wheel.dae" />
+                    <mesh filename="package://limo_description/meshes/limo_wheel.dae" scale="2 2 2" />
                 </geometry>
             </visual>
@@ -43,5 +43,5 @@
                 <origin xyz="0 0 0" rpy="0 0 0"/>
                 <geometry>
-                    <cylinder radius="0.02" length="0.01"/>
+                    <cylinder radius="0.04" length="0.02"/>
                 </geometry>
                 <material name='laser_material'>
@@ -55,5 +55,5 @@
                 <origin xyz="0 0 0" rpy="0 0 0"/>
                 <geometry>
-                    <cylinder radius="0.032" length="0.016"/>
+                    <cylinder radius="0.064" length="0.032"/>
                 </geometry>
             </collision>
@@ -83,5 +83,5 @@
                 <origin xyz="0 0 0" rpy="0 0 0"/>
                 <geometry>
-                    <box size="0.02 0.06 0.015"/>
+                    <box size="0.04 0.12 0.03"/>
                 </geometry>
                 <material name='depth_camera_material'>
@@ -95,5 +95,5 @@
                 <origin xyz="0 0 0" rpy="0 0 0"/>
                 <geometry>
-                    <box size="0.02 0.06 0.015"/>
+                    <box size="0.04 0.12 0.03"/>
                 </geometry>
             </collision>
@@ -129,5 +129,5 @@
                 <origin xyz="0 0 0" rpy="0 0 0"/>
                 <geometry>
-                    <box size="0.001 0.001 0.001"/>
+                    <box size="0.002 0.002 0.002"/>
                 </geometry>
                 <material name='imu_material'>
@@ -141,5 +141,5 @@
                 <origin xyz="0 0 0" rpy="0 0 0"/>
                 <geometry>
-                    <box size="0.001 0.001 0.001"/>
+                    <box size="0.002 0.002 0.002"/>
                 </geometry>
             </collision>
